File: BF-AVR/BF-AVR.kicad_sch (KiCad schematic)
At the start: 22 parts, among them J1 USB_B, Q1 NPN, Q2 NPN, Q3 NPN, U1 ATmega328P IO, U2 ATmega328P CPU, U3 ATmega328P PPU, Y1 16MHz, Y2 16MHz, Y3 16MHz

Commit message: a
Parts:
- removed C1: 1μF, symbol Device:C
- removed C4, C5, C8, C9: 22pF, symbol Device:C
- removed Q1, Q2, Q3: NPN, symbol Simulation_SPICE:NPN
- removed R1, R2, R3: 10kΩ, symbol Device:R
- removed U1: ATmega328P IO, Package_DIP:DIP-28_W7.62mm, symbol MCU_Microchip_ATmega:ATmega328P-P
- removed U2: ATmega328P CPU, Package_DIP:DIP-28_W7.62mm, symbol MCU_Microchip_ATmega:ATmega328P-P
- removed U3: ATmega328P PPU, Package_DIP:DIP-28_W7.62mm, symbol MCU_Microchip_ATmega:ATmega328P-P
- removed Y1, Y3: 16MHz, symbol Device:Crystal
- added U2: ATmega1284P PPU, Package_DIP:DIP-40_W15.24mm, symbol MCU_Microchip_ATmega:ATmega1284P-P
- C2, C3: value 1μF -> 0.1μF
Connections:
- net GND: now also U2.11 (GND), U2.31 (GND)
- net VCC: now also U2.10 (VCC), U2.30 (AVCC)
- net at C6.1, Y2.1: now also U2.13 (XTAL1)
- net at C7.1, Y2.2: now also U2.12 (XTAL2)
- no-connect marks 5 -> 2
